File: lowerBoard.sch (KiCad schematic (older format))
At the start: 34 parts, among them J1 Board->Board, J2 Drop_Header, J3 Debug, J4 Can_Bus, J5 LED, Q1 BSN20, Q2 BSN20, U1 STM32F407VGTx, U2 SN65HVD232, U3 MC34063AD

Commit message: Add files via upload
Parts:
- removed J1: Board->Board, Connector_Molex:Molex_KK-254_AE-6410-10A_1x10_P2.54mm_Vertical, symbol Connector:Conn_01x10_Female
- removed J5: LED, symbol Connector:Conn_01x04_Female
- removed Q1, Q2: BSN20, Package_TO_SOT_SMD:SOT-23, symbol Transistor_FET:BSN20
- removed R1: 0.75ohm, Resistor_SMD:R_0805_2012Metric_Pad1.15x1.40mm_HandSolder, symbol Device:R_Small
- removed R2: 11k, Resistor_SMD:R_0805_2012Metric_Pad1.15x1.40mm_HandSolder, symbol Device:R_Small
- removed R3: 18k, Resistor_SMD:R_0805_2012Metric_Pad1.15x1.40mm_HandSolder, symbol Device:R_Small
- removed R4: 300ohm, symbol Device:R_Small
- removed R5: 300ohm, Resistor_SMD:R_0805_2012Metric_Pad1.15x1.40mm_HandSolder, symbol Device:R_Small
- added C16, C17: 0.1 uF, Capacitor_SMD:C_0603_1608Metric, symbol Device:C_Small
- added H1, H2, H3: MountingHole_Pad, MountingHole:MountingHole_3mm_Pad_Via, symbol Mechanical:MountingHole_Pad
- added J1: LED_Header, Connector_Molex:Molex_KK-254_AE-6410-05A_1x05_P2.54mm_Vertical, symbol Connector:Conn_01x05_Male
- added J6: Board -> Board, Connector_Molex:Molex_KK-254_AE-6410-11A_1x11_P2.54mm_Vertical, symbol Connector:Conn_01x11_Male
- added Q1, Q2: IRLML0030, Package_TO_SOT_SMD:SOT-23, symbol Transistor_FET:IRLML0030
- added R1: 0.75 Ω, Resistor_SMD:R_0603_1608Metric, symbol Device:R_Small_US
- added R10, R7: 2 Ω, Resistor_SMD:R_0603_1608Metric, symbol Device:R_Small_US
- added R11, R12, R6, R9: 10 kΩ, Resistor_SMD:R_0603_1608Metric, symbol Device:R_Small_US
- added R2: 11 kΩ, Resistor_SMD:R_0603_1608Metric, symbol Device:R_Small_US
- added R3: 18 kΩ, Resistor_SMD:R_0603_1608Metric, symbol Device:R_Small_US
- added R4: 120 Ω, Resistor_SMD:R_0603_1608Metric, symbol Device:R_Small_US
- added R5, R8: 1 kΩ, Resistor_SMD:R_0603_1608Metric, symbol Device:R_Small_US
- added SW1, SW2: SW_Push, Button_Switch_SMD:SW_SPST_B3S-1000, symbol Switch:SW_Push
- C1, C10, C11, C12, C14, C2, C4, C5, C6, C7, C8, C9: footprint Capacitor_SMD:C_0805_2012Metric_Pad1.15x1.40mm_HandSolder -> Capacitor_SMD:C_0603_1608Metric
- C13, C15: footprint Capacitor_SMD:C_Elec_10x10.2 -> Capacitor_SMD:C_0603_1608Metric
- C3: footprint (none) -> Capacitor_SMD:C_0603_1608Metric
- D1: footprint Diode_THT:D_5W_P10.16mm_Horizontal -> Diode_SMD:D_0603_1608Metric
- L1: footprint Inductor_THT:L_Axial_L20.3mm_D12.1mm_P28.50mm_Horizontal_Vishay_IHA-101 -> Capacitor_SMD:C_0603_1608Metric
Connections:
- net +3V3: now also J6.11 (Pin_11), R11.1, R12.1, R3.1
- net BATT_IN: now also J2.2 (Pin_2), J6.10 (Pin_10), R1.2
- net CAN_H: now also R4.1
- net CAN_L: now also R4.2
- net CS_Accel: now also J6.5 (Pin_5)
- net Drop: now also J6.9 (Pin_9), R10.1; no longer J2.1 (Pin_1)
- net Drop_Signal: now also R8.2
- net GND: now also U1.94 (BOOT0), C16.1, C17.1, H1.1, H2.1, H3.1, J1.1 (Pin_1), J6.1 (Pin_1), Q1.2 (S), Q2.2 (S), R2.2, R6.1, R9.1, SW1.1, SW2.1; no longer J2.2 (Pin_2)
- net Ignite: now also J2.1 (Pin_1), R7.1
- net Ignite_Signal: now also R5.2
- net LED1: now also J1.5 (Pin_5)
- net LED2: now also J1.4 (Pin_4)
- net LED3: now also J1.3 (Pin_3)
- net LED4: now also J1.2 (Pin_2)
- net RX: now also J6.7 (Pin_7)
- net SCLK: now also J6.2 (Pin_2)
- net SDI: now also J6.3 (Pin_3)
- net SDO: now also J6.4 (Pin_4)
- net TX: now also J6.8 (Pin_8)
- net RESET: now reaches U1.14 (NRST)
- net RESET: now also C16.2, R12.2, SW1.2
- net ARM: now reaches U1.51 (PB12)
- net ARM: now also C17.2, R11.2, SW2.2
- net at U3.1 (SwC), U3.7 (Ipk), U3.8 (DC): now also R1.1
- net at U3.5 (Vfb): now also R2.1, R3.2
- net CS_Barrom renamed CS_Baro
- net CS_Baro: now also J6.6 (Pin_6)
- new net: Q1.1 (G), R5.1, R6.2
- new net: Q1.3 (D), R7.2
- new net: Q2.1 (G), R8.1, R9.2
- new net: Q2.3 (D), R10.2
- no-connect marks 67 -> 64
Other:
- note added: "18650 Li-Ion Cells\n"
- note added: "8.4 -> 3.3 V Buck"
- note added: "ARM Button\n"
- note added: "CAN Transciever"
- note added: "I/O Headers"
- note added: "Ignition Power MOSFET"
- note added: "MCU RESET Button\n"
- note added: "Release Power MOSFET"
- note added: "Todo:\nAdd arm button\nAdd reset button\nCreate footprint for new FETS\nSPICE it up\nChange everything to 0603"
- moved on the sheet: BT1, BT2, C12, C13, C14, C15, D1, J2, J3, J4, L1, U2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
