File: upperBoard.sch (KiCad schematic (older format))
At the start: 10 parts, among them IC1 FGPMMOPA6H, J1 Board->Board, J2 Ignite_Header, U1 ICM-20948, U2 MS5607-02BA

Commit message: Added routed upper board files
Parts:
- added H1, H2, H3, H4: MountingHole_Pad, MountingHole:MountingHole_3mm_Pad_Via, symbol Mechanical:MountingHole_Pad
Connections:
- net GND: now also H1.1, H2.1, H3.1, H4.1
Changed lines of the file:
@@
 	1    0    0    -1
 $EndComp
+$Comp
+L Mechanical:MountingHole_Pad H2
+U 1 1 5E4B8D6F
+P 2100 1250
+F 0 "H2" H 2200 1299 50  0000 L CNN
+F 1 "MountingHole_Pad" H 2200 1208 50  0000 L CNN
+F 2 "MountingHole:MountingHole_3mm_Pad_Via" H 2100 1250 50  0001 C CNN
+F 3 "~" H 2100 1250 50  0001 C CNN
+	1    2100 1250
+	1    0    0    -1
+$EndComp
+$Comp
+L Mechanical:MountingHole_Pad H3
+U 1 1 5E4BB0CA
+P 2100 2150
+F 0 "H3" H 2200 2199 50  0000 L CNN
+F 1 "MountingHole_Pad" H 2200 2108 50  0000 L CNN
+F 2 "MountingHole:MountingHole_3mm_Pad_Via" H 2100 2150 50  0001 C CNN
+F 3 "~" H 2100 2150 50  0001 C CNN
+	1    2100 2150
+	-1   0    0    1
+$EndComp
+$Comp
+L Mechanical:MountingHole_Pad H1
+U 1 1 5E4BC498
+P 1750 1700
+F 0 "H1" H 1850 1749 50  0000 L CNN
+F 1 "MountingHole_Pad" H 1850 1658 50  0000 L CNN
+F 2 "MountingHole:MountingHole_3mm_Pad_Via" H 1750 1700 50  0001 C CNN
+F 3 "~" H 1750 1700 50  0001 C CNN
+	1    1750 1700
+	0    -1   -1   0
+$EndComp
+$Comp
+L Mechanical:MountingHole_Pad H4
+U 1 1 5E4BD731
+P 2500 1750
+F 0 "H4" H 2600 1799 50  0000 L CNN
+F 1 "MountingHole_Pad" H 2600 1708 50  0000 L CNN
+F 2 "MountingHole:MountingHole_3mm_Pad_Via" H 2500 1750 50  0001 C CNN
+F 3 "~" H 2500 1750 50  0001 C CNN
+	1    2500 1750
+	0    1    1    0
+$EndComp
+$Comp
+L power:GND #PWR0103
+U 1 1 5E4BE57D
+P 2100 1700
+F 0 "#PWR0103" H 2100 1450 50  0001 C CNN
+F 1 "GND" H 2105 1527 50  0000 C CNN
+F 2 "" H 2100 1700 50  0001 C CNN
+F 3 "" H 2100 1700 50  0001 C CNN
+	1    2100 1700
+	1    0    0    -1
+$EndComp
+Wire Wire Line
+	2100 2050 2400 2050
+Wire Wire Line
+	2400 2050 2400 1750
+Wire Wire Line
+	2400 1750 2400 1700
+Wire Wire Line
+	2400 1700 2100 1700
+Connection ~ 2400 1750
+Wire Wire Line
+	2100 1700 2100 1350
+Connection ~ 2100 1700
+Wire Wire Line
+	2100 1700 1850 1700
 $EndSCHEMATC

Commit message: Add files via upload
Parts:
- removed J1: Board->Board, Connector_Molex:Molex_KK-254_AE-6410-10A_1x10_P2.54mm_Vertical, symbol Connector:Conn_01x10_Female
- added J1: Conn_01x11_Male, Connector_Molex:Molex_KK-254_AE-6410-11A_1x11_P2.54mm_Vertical, symbol Connector:Conn_01x11_Male
- J2: value Ignite_Header -> Release_Header
Connections:
- net +3V3: now also J1.11 (Pin_11)
- net CS_Accel: now also J1.5 (Pin_5)
- net CS_Barrom: now also J1.6 (Pin_6)
- net GND: now also J1.1 (Pin_1); no longer J2.2 (Pin_2)
- net RX: now also J1.7 (Pin_7)
- net SCLK: now also J1.2 (Pin_2)
- net SDI: now also J1.3 (Pin_3)
- net SDO: now also J1.4 (Pin_4)
- net TX: now also J1.8 (Pin_8)
- net Ignite renamed Release
- net Release: now also J1.9 (Pin_9)
- new net Release_Return: J1.10 (Pin_10), J2.2 (Pin_2)
Changed lines of the file:
@@
 L power:PWR_FLAG #FLG0101
 U 1 1 5E36079F
-P 5400 4550
-F 0 "#FLG0101" H 5400 4625 50  0001 C CNN
-F 1 "PWR_FLAG" V 5400 4677 50  0000 L CNN
-F 2 "" H 5400 4550 50  0001 C CNN
-F 3 "~" H 5400 4550 50  0001 C CNN
-	1    5400 4550
+P 5100 4450
+F 0 "#FLG0101" H 5100 4525 50  0001 C CNN
+F 1 "PWR_FLAG" V 5100 4577 50  0000 L CNN
+F 2 "" H 5100 4450 50  0001 C CNN
+F 3 "~" H 5100 4450 50  0001 C CNN
+	1    5100 4450
 	0    -1   -1   0
 $EndComp
@@
 L power:+3.3V #PWR0101
 U 1 1 5E354748
-P 5400 4550
-F 0 "#PWR0101" H 5400 4400 50  0001 C CNN
-F 1 "+3.3V" H 5415 4723 50  0000 C CNN
-F 2 "" H 5400 4550 50  0001 C CNN
-F 3 "" H 5400 4550 50  0001 C CNN
-	1    5400 4550
+P 5100 4450
+F 0 "#PWR0101" H 5100 4300 50  0001 C CNN
+F 1 "+3.3V" H 5115 4623 50  0000 C CNN
+F 2 "" H 5100 4450 50  0001 C CNN
+F 3 "" H 5100 4450 50  0001 C CNN
+	1    5100 4450
 	1    0    0    -1
 $EndComp
@@
 Text Label 5400 4750 0    50   ~ 0
 TX
-$Comp
-L Connector:Conn_01x10_Female J1
-U 1 1 5E34D348
-P 6050 4950
-F 0 "J1" H 6078 4926 50  0000 L CNN
-F 1 "Board->Board" H 6078 4835 50  0000 L CNN
-F 2 "Connector_Molex:Molex_KK-254_AE-6410-10A_1x10_P2.54mm_Vertical" H 6050 4950 50  0001 C CNN
-F 3 "~" H 6050 4950 50  0001 C CNN
-	1    6050 4950
-	1    0    0    -1
-$EndComp
-Wire Wire Line
-	5850 4550 5400 4550
 Wire Wire Line
 	5850 4750 5400 4750
@@
 Wire Wire Line
 	5850 5350 5400 5350
-Connection ~ 5400 4550
-Wire Wire Line
-	5850 4650 5400 4650
+Connection ~ 5100 4450
 Text Label 5400 4650 0    50   ~ 0
-Ignite
+Release
 $Comp
 L Connector:Conn_01x02_Female J2
@@
 P 6050 5950
 F 0 "J2" H 6078 5926 50  0000 L CNN
-F 1 "Ignite_Header" H 6078 5835 50  0000 L CNN
+F 1 "Release_Header" H 6078 5835 50  0000 L CNN
 F 2 "Connector_Molex:Molex_KK-254_AE-6410-02A_1x02_P2.54mm_Vertical" H 6050 5950 50  0001 C CNN
 F 3 "~" H 6050 5950 50  0001 C CNN
@@
 Wire Wire Line
 	5850 5950 5550 5950
-Text Label 5550 5950 0    50   ~ 0
-Ignite
-$Comp
-L power:GND #PWR015
-U 1 1 5E37E9BA
-P 5550 6050
-F 0 "#PWR015" H 5550 5800 50  0001 C CNN
-F 1 "GND" H 5555 5877 50  0000 C CNN
-F 2 "" H 5550 6050 50  0001 C CNN
-F 3 "" H 5550 6050 50  0001 C CNN
-	1    5550 6050
-	1    0    0    -1
-$EndComp
-Wire Wire Line
-	5550 6050 5850 6050
 Wire Wire Line
 	5400 5450 5700 5450
@@
 Wire Wire Line
 	2100 1700 1850 1700
+$Comp
+L Connector:Conn_01x11_Male J1
+U 1 1 5E5632B6
+P 6050 4950
+F 0 "J1" H 6158 5631 50  0000 C CNN
+F 1 "Conn_01x11_Male" H 6158 5540 50  0000 C CNN
+F 2 "Connector_Molex:Molex_KK-254_AE-6410-11A_1x11_P2.54mm_Vertical" H 6050 4950 50  0001 C CNN
+F 3 "~" H 6050 4950 50  0001 C CNN
+	1    6050 4950
+	-1   0    0    1
+$EndComp
+Wire Wire Line
+	5100 4450 5850 4450
+Text Label 5300 4550 0    50   ~ 0
+Release_Return
+Wire Wire Line
+	5300 4550 5850 4550
+Wire Wire Line
+	5850 4650 5400 4650
+Text Label 5550 5950 0    50   ~ 0
+Release
+Text Label 5250 6050 0    50   ~ 0
+Release_Return
+Wire Wire Line
+	5250 6050 5850 6050
 $EndSCHEMATC
